File: fpga_adapter.kicad_pcb (KiCad board)
At the start: 2 copper layers, 105.1 x 49.2 mm, 4 parts, among them J1 Conn_02x25_Counter_Clockwise, J2 Conn_02x03_Counter_Clockwise, J3 Conn_02x03_Counter_Clockwise, X1 SHC-68

Commit message: finished routing
Parts:
- removed J1: Conn_02x25_Counter_Clockwise, Connector_IDC:IDC-Header_2x25-1MP_P2.54mm_Latch12.0mm_Vertical
- removed J2, J3: Conn_02x03_Counter_Clockwise, Connector_Molex:Molex_Mini-Fit_Jr_5569-06A2_2x03_P4.20mm_Horizontal
- added PWR0: Conn_02x03_Top_Bottom, Connector_Molex:Molex_Mini-Fit_Jr_5569-06A2_2x03_P4.20mm_Horizontal, F.Cu at (174.3, 131.1)
- added PWR1: Conn_02x03_Top_Bottom, Connector_Molex:Molex_Mini-Fit_Jr_5569-06A2_2x03_P4.20mm_Horizontal, F.Cu at (191.2, 131.1)
- added X1: Conn_02x25_Odd_Even, Connector_IDC:IDC-Header_2x25-1MP_P2.54mm_Latch_Vertical, F.Cu at (122.9, 157.2)
- renumbered X1 to X0
Connections:
- X0 pad 10: Net-(X1-Pad10) -> /DIO8
- X0 pad 11: Net-(X1-Pad11) -> /DIO10
- X0 pad 12: Net-(X1-Pad12) -> /DIO12
- X0 pad 13: Net-(X1-Pad13) -> /DIO14
- X0 pad 14: Net-(X1-Pad14) -> /AGND
- X0 pad 15: Net-(X1-Pad15) -> /AGND
- X0 pad 16: Net-(X1-Pad16) -> /AGND
- X0 pad 17: Net-(X1-Pad17) -> /AGND
- X0 pad 18: Net-(X1-Pad18) -> /AGND
- X0 pad 19: Net-(X1-Pad19) -> /AGND
- X0 pad 2: Net-(X1-Pad2) -> /DGND
- X0 pad 20: Net-(X1-Pad20) -> /AGND
- X0 pad 21: Net-(X1-Pad21) -> /AGND
- X0 pad 24: Net-(X1-Pad24) -> /AGND
- X0 pad 27: Net-(X1-Pad27) -> /AGND
- X0 pad 29: Net-(X1-Pad29) -> /AI3N
- X0 pad 3: Net-(X1-Pad3) -> /DGND
- X0 pad 30: Net-(X1-Pad30) -> /AGND
- X0 pad 31: Net-(X1-Pad31) -> /AI2N
- X0 pad 32: Net-(X1-Pad32) -> /AI1N
- X0 pad 33: Net-(X1-Pad33) -> /AGND
- X0 pad 34: Net-(X1-Pad34) -> /AI0N
- X0 pad 36: Net-(X1-Pad36) -> /DIO0
- X0 pad 37: Net-(X1-Pad37) -> /DIO1
- X0 pad 38: Net-(X1-Pad38) -> /DIO2
- X0 pad 39: Net-(X1-Pad39) -> /DIO3
- X0 pad 4: Net-(X1-Pad4) -> /DGND
- X0 pad 40: Net-(X1-Pad40) -> /DIO4
- X0 pad 41: Net-(X1-Pad41) -> /DIO5
- X0 pad 42: Net-(X1-Pad42) -> /DIO6
- X0 pad 43: Net-(X1-Pad43) -> /DIO7
- X0 pad 44: Net-(X1-Pad44) -> /DIO9
- X0 pad 45: Net-(X1-Pad45) -> /DIO11
- X0 pad 46: Net-(X1-Pad46) -> /DIO13
- X0 pad 47: Net-(X1-Pad47) -> /DIO15
- X0 pad 5: Net-(X1-Pad5) -> /DGND
- X0 pad 54: Net-(X1-Pad54) -> /AO1
- X0 pad 55: Net-(X1-Pad55) -> /AO0
- X0 pad 58: Net-(X1-Pad58) -> /AGND
- X0 pad 6: Net-(X1-Pad6) -> /DGND
- X0 pad 61: Net-(X1-Pad61) -> /AGND
- X0 pad 63: Net-(X1-Pad63) -> /AI3P
- X0 pad 64: Net-(X1-Pad64) -> /AGND
- X0 pad 65: Net-(X1-Pad65) -> /AI2P
- X0 pad 66: Net-(X1-Pad66) -> /AI1P
- X0 pad 67: Net-(X1-Pad67) -> /AGND
- X0 pad 68: Net-(X1-Pad68) -> /AI0P
- X0 pad 7: Net-(X1-Pad7) -> /DGND
- X0 pad 8: Net-(X1-Pad8) -> /DGND
- X0 pad 9: Net-(X1-Pad9) -> /DGND
Routing:
- net /VCC3: track 0.00 -> 46.7 mm
- net /VCC1: track 0.00 -> 42.5 mm
- net /AI3P: track 0.00 -> 39.9 mm
- net /AI2P: track 0.00 -> 39.9 mm
- net /DIO0: track 0.00 -> 39.4 mm
- net /AI1P: track 0.00 -> 39.4 mm
- net /AI0P: track 0.00 -> 39.4 mm
- net /DIO1: track 0.00 -> 38.9 mm
- net /DIO2: track 0.00 -> 38.4 mm
- net /DIO15: track 0.00 -> 38.1 mm
- net /DIO3: track 0.00 -> 37.8 mm
- net /DIO13: track 0.00 -> 37.6 mm
- net /AI3N: track 0.00 -> 37.5 mm, vias 0 -> 1
- net /AI2N: track 0.00 -> 37.4 mm, vias 0 -> 1
- net /DIO4: track 0.00 -> 37.3 mm
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- added copper zone on B.Cu, net /AGND
- added copper zone on F.Cu, net /AGND
- added copper zone on F.Cu, net /DGND
Other:
- net class Default: clearance 0.2 -> 0.125; trace_width 0.25 -> 0.2; via_dia 0.8 -> 0.6; via_drill 0.4 -> 0.3
- net class pwr added: clearance 0.125, trace_width 1, via_dia 0.6, via_drill 0.3
- rule trace_clearance: 0.2 -> 0.125
- rule trace_min: 0.2 -> 0.125
