File: fpga_adapter.sch (KiCad schematic (older format))
At the start: 4 parts, among them J1 Conn_02x25_Counter_Clockwise, J2 Conn_02x03_Counter_Clockwise, J3 Conn_02x03_Counter_Clockwise, X1 SHC-68

Commit message: finished routing
Parts:
- removed J1: Conn_02x25_Counter_Clockwise, Connector_IDC:IDC-Header_2x25-1MP_P2.54mm_Latch12.0mm_Vertical, symbol Connector_Generic:Conn_02x25_Counter_Clockwise
- removed J2, J3: Conn_02x03_Counter_Clockwise, Connector_Molex:Molex_Mini-Fit_Jr_5569-06A2_2x03_P4.20mm_Horizontal, symbol Connector_Generic:Conn_02x03_Counter_Clockwise
- added PWR0, PWR1: Conn_02x03_Top_Bottom, Connector_Molex:Molex_Mini-Fit_Jr_5569-06A2_2x03_P4.20mm_Horizontal, symbol Connector_Generic:Conn_02x03_Top_Bottom
- added X1: Conn_02x25_Odd_Even, Connector_IDC:IDC-Header_2x25-1MP_P2.54mm_Latch_Vertical, symbol Connector_Generic:Conn_02x25_Odd_Even
- X0: renamed from X1; symbol spels_dev:SHC-68 -> fpga_adapter-rescue:SHC-68-spels_dev
Connections:
- net CLKOUT is gone; now on net AGND: X0.33 (P33)
- net P0.5 is gone; now on net AGND: X0.27 (P27)
- net P1.3 is gone; now on net AGND: X0.21 (P21)
- net P1.5 is gone; now on net AGND: X0.19 (P19)
- net P1.7 is gone; now on net AGND: X0.17 (P17)
- net P2.1 is gone; now on net AGND: X0.15 (P15)
- net PFI3 is gone; now on net AGND: X0.30 (P30)
- net DIO0: now reaches X0.36 (P36)
- net DIO0: now also X1.33 (Pin_33)
- net DIO1: now reaches X0.37 (P37)
- net DIO1: now also X1.31 (Pin_31)
- net DIO2: now reaches X0.38 (P38)
- net DIO2: now also X1.29 (Pin_29)
- net DIO3: now reaches X0.39 (P39)
- net DIO3: now also X1.27 (Pin_27)
- net DIO4: now reaches X0.40 (P40)
- net DIO4: now also X1.25 (Pin_25)
- net DIO5: now reaches X0.41 (P41)
- net DIO5: now also X1.23 (Pin_23)
- net DIO6: now reaches X0.42 (P42)
- net DIO6: now also X1.21 (Pin_21)
- net DIO7: now reaches X0.43 (P43)
- net DIO7: now also X1.19 (Pin_19)
- net DIO9: now reaches X0.44 (P44)
- net DIO9: now also X1.17 (Pin_17)
- net DIO11: now reaches X0.45 (P45)
- net DIO11: now also X1.15 (Pin_15)
- net DIO13: now reaches X0.46 (P46)
- net DIO13: now also X1.13 (Pin_13)
- net DIO15: now reaches X0.47 (P47)
- net DIO15: now also X1.11 (Pin_11)
- net AO1: now reaches X0.54 (P54)
- net AO1: now also X1.10 (Pin_10)
- net AO0: now reaches X0.55 (P55)
- net AO0: now also X1.9 (Pin_9)
- net AGND: now reaches X0.58 (P58)
- net AGND: now also X0.14 (P14), X0.16 (P16), X0.18 (P18), X0.20 (P20), X0.24 (P24), X0.61 (P61), X0.64 (P64), X0.67 (P67), X1.12 (Pin_12), X1.14 (Pin_14), X1.16 (Pin_16), X1.18 (Pin_18)
- net AI3P: now reaches X0.63 (P63)
- net AI3P: now also X1.7 (Pin_7)
- net AI2P: now reaches X0.65 (P65)
- net AI2P: now also X1.5 (Pin_5)
- net AI1P: now reaches X0.66 (P66)
- net AI1P: now also X1.3 (Pin_3)
- net AI0P: now reaches X0.68 (P68)
- net AI0P: now also X1.1 (Pin_1)
- removed net GND: X0.10 (P10), X0.12 (P12), X0.14 (P14), X0.16 (P16), X0.18 (P18), X0.2 (P2), X0.20 (P20), X0.22 (P22), X0.24 (P24), X0.28 (P28), X0.32 (P32), X0.34 (P34), X0.4 (P4), X0.6 (P6), X0.8 (P8)
- net P0.1 renamed AI2N
- net AI2N: now also X1.6 (Pin_6)
- net P0.3 renamed AI3N
- net AI3N: now also X1.8 (Pin_8)
- net P0.7: no longer names the net of X0.25 (P25)
- net P1.1: no longer names the net of X0.23 (P23)
- net P2.3 renamed DIO14
- net DIO14: now also X1.20 (Pin_20)
- net P2.5 renamed DIO10
- net DIO10: now also X1.24 (Pin_24)
- net P2.7 renamed DGND
- net DGND: now also X0.2 (P2), X0.3 (P3), X0.4 (P4), X0.5 (P5), X0.6 (P6), X0.7 (P7), X0.8 (P8), X1.28 (Pin_28), X1.30 (Pin_30), X1.32 (Pin_32), X1.34 (Pin_34)
- net PFI1: no longer names the net of X0.26 (P26)
- removed net RESERVED: X0.1 (P1), X0.3 (P3), X0.5 (P5), X0.7 (P7)
- new net AI0N: X0.34 (P34), X1.2 (Pin_2)
- new net AI1N: X0.32 (P32), X1.4 (Pin_4)
- new net DIO12: X0.12 (P12), X1.22 (Pin_22)
- new net DIO8: X0.10 (P10), X1.26 (Pin_26)
- new net PWGND0: PWR0.4 (Pin_4), X1.37 (Pin_37), X1.38 (Pin_38)
- new net PWGND1: PWR0.5 (Pin_5), X1.39 (Pin_39), X1.40 (Pin_40)
- new net PWGND2: PWR1.4 (Pin_4), X1.45 (Pin_45), X1.46 (Pin_46)
- new net PWGND3: PWR1.5 (Pin_5), X1.47 (Pin_47), X1.48 (Pin_48)
- new net VCC0: PWR0.1 (Pin_1), X1.35 (Pin_35), X1.36 (Pin_36)
- new net VCC1: PWR0.2 (Pin_2), X1.41 (Pin_41), X1.42 (Pin_42)
- new net VCC2: PWR1.1 (Pin_1), X1.43 (Pin_43), X1.44 (Pin_44)
- new net VCC3: PWR1.2 (Pin_2), X1.49 (Pin_49), X1.50 (Pin_50)
- no-connect marks 0 -> 22
Other:
- moved on the sheet: X0
